Commit message: fix(vs050): correct tool0 frame orientation math and indentation
- Remove the incorrect `radians()` function wrapper around `pi` in the `J6-tool0` joint origin. Since `pi` is already in radians, `radians(pi)` resulted in an incorrect rotation.
- Fix XML indentation for the child, parent, and origin tags within the flange and tool0 joints to improve code readability.

File: denso_robot_descriptions/robots/vs050/urdf/denso_robot_kinematics.xacro (robot description, xacro)
@@ -193,13 +193,13 @@
 		<link name="${namespace}flange"/>
 		<joint name="${namespace}J6-flange" type="fixed">
-		<parent link="${namespace}J6"/>
-		<child link="${namespace}flange"/>
-		<origin rpy="0 0 0" xyz="0 0 0"/>
+			<parent link="${namespace}J6"/>
+			<child link="${namespace}flange"/>
+			<origin rpy="0 0 0" xyz="0 0 0"/>
 		</joint>
 		<link name="${namespace}tool0"/>
 		<joint name="${namespace}J6-tool0" type="fixed">
-		<parent link="${namespace}J6"/>
-		<child link="${namespace}tool0"/>
-		<origin rpy="${radians(pi)} ${radians(-pi/2)} 0" xyz="0 0 0"/>
+			<parent link="${namespace}J6"/>
+			<child link="${namespace}tool0"/>
+			<origin rpy="${pi} ${-pi/2} 0" xyz="0 0 0"/>
 		</joint>
 	</xacro:macro>
